File: Controller/controller.sch (KiCad schematic (older format))
At the start: 62 parts, among them IC1 ATMEGA8-AI, IC2 MOC3042M, J1 USB, P1 CONN_4, P10 CONN_2, P11 CONN_2, P12 NTC, P13 CONN_5, P2 CONN_1, P3 CONN_1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

Commit message: Cosmetic changes
Parts:
- C1, C10, C11, C12, C13, C2, C3, C4, C5, C6, C7, C8, C9: symbol C -> C-RESCUE-controller
- D2, D5: symbol LED -> LED-RESCUE-controller
- D3, D4: symbol ZENER -> ZENER-RESCUE-controller
- IC2: symbol MOC3042M -> MOC3042M-RESCUE-controller
- R1, R10, R11, R12, R13, R14, R15, R16, R17, R2, R27, R28, R29, R3, R4, R5, R6, R7, R8, R9: symbol R -> R-RESCUE-controller
Other:
- moved on the sheet: C10, C11, C6, C7, C9, D6, P10, P12, Q1, R11, R12, R13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
